Commit message: fix kin

File: adeept_description/urdf/adeept_description.xacro (robot description, xacro)
@@ -291,5 +291,5 @@
       friction="0.1" />
   </joint>
-    <link
+  <link
     name="end">
     <inertial>
@@ -298,12 +298,12 @@
         rpy="0 0 0" />
       <mass
-        value="0.001" />
-      <inertia
-        ixx="4E-10"
-        ixy="0"
-        ixz="0"
-        iyy="4E-10"
-        iyz="0"
-        izz="4E-10" />
+        value="0.01" />
+      <inertia
+        ixx="4E-5"
+        ixy="0"
+        ixz="0"
+        iyy="4E-5"
+        iyz="0"
+        izz="4E-5" />
     </inertial>
     <visual>
@@ -327,5 +327,5 @@
   <joint
     name="Joint_end"
-    type="fixed">
+    type="prismatic">
     <origin
       xyz="0.013 0 0.0665"
@@ -337,4 +337,12 @@
     <axis
       xyz="0 0 1" />
+    <limit
+      lower="0"
+      upper="0"
+      effort="100.0"
+      velocity="0.5" />
+    <dynamics
+      damping="0.2"
+      friction="0.1" />
   </joint>
   <!-- Controller -->

Commit message: add_pen

File: adeept_description/urdf/adeept_description.xacro (robot description, xacro)
@@ -292,5 +292,5 @@
   </joint>
   <link
-    name="end">
+    name="pen">
     <inertial>
       <origin
@@ -309,22 +309,22 @@
     <visual>
       <origin
-        xyz="0 0 0"
-        rpy="0 0 0" />
-      <geometry>
-        <sphere radius = "0.001"/>
-      </geometry>
-      <material name = "black"/>
-    </visual>
-    <collision>
-      <origin
-        xyz="0 0 0"
-        rpy="0 0 0" />
-      <geometry>
-        <sphere radius = "0.001"/>
-      </geometry>
-    </collision>
-  </link>
-  <joint
-    name="Joint_end"
+        xyz="0.02 0 0"
+        rpy="0 1.5707 0" />
+      <geometry>
+        <cylinder radius = "0.003" length="0.2"/>
+      </geometry>
+      <material name = "brown"/>
+    </visual>
+    <collision>
+      <origin
+        xyz="0.027 0 0"
+        rpy="0 1.5707 0" />
+      <geometry>
+        <cylinder radius = "0.003" length="0.2"/>
+      </geometry>
+    </collision>
+  </link>
+  <joint
+    name="Joint_pen"
     type="prismatic">
     <origin
@@ -333,4 +333,57 @@
     <parent
       link="Link_4" />
+    <child
+      link="pen" />
+    <limit
+      lower="0"
+      upper="0"
+      effort="100.0"
+      velocity="1.0" />
+    <dynamics
+      damping="0.2"
+      friction="0.1" />
+  </joint>
+    <link
+    name="end">
+    <inertial>
+      <origin
+        xyz="0 0 0"
+        rpy="0 0 0" />
+      <mass
+        value="0.001" />
+      <inertia
+        ixx="4E-2"
+        ixy="0"
+        ixz="0"
+        iyy="4E-2"
+        iyz="0"
+        izz="4E-2" />
+    </inertial>
+    <visual>
+      <origin
+        xyz="0 0 0"
+        rpy="0 0 0" />
+      <geometry>
+        <sphere radius = "0.001"/>
+      </geometry>
+      <material name = "black"/>
+    </visual>
+    <collision>
+      <origin
+        xyz="0 0 0"
+        rpy="0 0 0" />
+      <geometry>
+        <sphere radius = "0.001"/>
+      </geometry>
+    </collision>
+  </link>
+  <joint
+    name="pen_end"
+    type="prismatic">
+    <origin
+      xyz="0.12 0 0"
+      rpy="0 0 0" />
+    <parent
+      link="pen" />
     <child
       link="end" />
